File: PCB/PCB-V2/Miguel's-Custom-Devboard - V2.kicad_sch (KiCad schematic)
At the start: 36 parts, among them J1 USB_C_Receptacle_USB2.0_14P, J2 Conn_01x20, J3 Conn_01x20, J4 Conn_01x03, SW1 SW_Push, U1 RP2040, U2 MCP1700x-330xxTT, U3 W25Q16JVZPIQ TR, Y1 12 MHz

Commit message: m
Other:
- title: (none) -> Miguel's Custom Devboard
Changed lines of the file:
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@@
 	(generator_version "9.0")
 	(paper "A4")
+	(title_block
+		(title "Miguel's Custom Devboard")
+		(date "1/9/26")
+		(rev "V2")
+	)
 	(text_box "Crystal Oscillator"
 		(exclude_from_sim no)
