File: PCB/PCB-V2/Miguel's-Custom-Devboard - V2.kicad_pcb (KiCad board)
At the start: 2 copper layers, 21 x 51 mm, 36 parts, among them J1 USB_C_Receptacle_USB2.0_14P, J2 Conn_01x20, J3 Conn_01x20, J4 Conn_01x03, SW1 SW_Push, U1 RP2040, U2 MCP1700x-330xxTT, U3 W25Q16JVZPIQ TR, Y1 12 MHz

Commit message: Final Update
Parts:
- J2, J3, J4: moved to B.Cu
- turned J2 to 180 degrees
- turned J3 to 180 degrees
- turned J4 to -90 degrees
